Commit message: smoot run and multi robot

File: src/curobo/content/assets/robot/ridgeback_franka/RidgebackFranka1.urdf (robot description, URDF)
Before this commit: robot RidgebackFranka, 19 links, 18 joints
Links:
- link RidgebackFranka_panda_link3: geometry collision box size=0.001 0.001 0.001; visual mesh filename=meshes/RidgebackFranka_panda_link3_collisions.obj scale=1. 1. 1.
- link RidgebackFranka_panda_link4: geometry visual mesh filename=meshes/RidgebackFranka_panda_link4_collisions.obj scale=1. 1. 1.; visual mesh filename=meshes/RidgebackFranka_panda_link4_visuals_panda_link4.obj scale=0.01 0.01 0.01
- link RidgebackFranka_panda_link5: geometry visual mesh filename=meshes/RidgebackFranka_panda_link5_collisions.obj scale=1. 1. 1.; visual mesh filename=meshes/RidgebackFranka_panda_link5_visuals_panda_link5.obj scale=0.01 0.01 0.01
- link RidgebackFranka_panda_link6: geometry visual mesh filename=meshes/RidgebackFranka_panda_link6_collisions.obj scale=1. 1. 1.; visual mesh filename=meshes/RidgebackFranka_panda_link6_visuals_panda_link6.obj scale=0.01 0.01 0.01
- link RidgebackFranka_panda_link7: geometry visual mesh filename=meshes/RidgebackFranka_panda_link7_collisions.obj scale=1. 1. 1.; visual mesh filename=meshes/RidgebackFranka_panda_link7_visuals_panda_link7.obj scale=0.01 0.01 0.01
- link RidgebackFranka_panda_rightfinger: geometry visual mesh filename=meshes/RidgebackFranka_panda_rightfinger_collisions.obj scale=1. 1. 1.; visual mesh filename=meshes/RidgebackFranka_panda_rightfinger_visuals_panda_righ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 scale=0.01 0.01 0.01
- link dummy_base_x: mass 0.0001 -> 0.1
- link dummy_base_y: mass 0.0001 -> 0.1
Joints:
- joint dummy_base_prismatic_x_joint: limit lower=-600.2800293 upper=600.2800293 effort=4800. velocity=15. -> lower=-100.2800293 upper=100.2800293 effort=4800. velocity=15.
- joint dummy_base_prismatic_y_joint: limit lower=-600.2800293 upper=600.2800293 effort=4800. velocity=15. -> lower=-100.2800293 upper=100.2800293 effort=4800. velocity=15.
- joint dummy_base_revolute_z_joint: limit lower=-600.2800208 upper=600.2800208 effort=4800. velocity=15.0000002 -> lower=-100.2800208 upper=100.2800208 effort=4800. velocity=15.0000002
