Commit message: move smooth

File: src/curobo/content/assets/robot/ridgeback_franka/RidgebackFranka.urdf (robot description, URDF)
Before this commit: robot RidgebackFranka, 19 links, 18 joints
Links:
- link dummy_base_x: mass 0.0001 -> 0.1
- link dummy_base_y: mass 0.0001 -> 0.1

Commit message: good ik

File: src/curobo/content/assets/robot/ridgeback_franka/RidgebackFranka.urdf (robot description, URDF)
Before this commit: robot RidgebackFranka, 19 links, 18 joints
Joints:
- joint dummy_base_prismatic_x_joint: limit lower=-600.2800293 upper=600.2800293 effort=4800. velocity=15. -> lower=-100.2800293 upper=100.2800293 effort=4800. velocity=15.
- joint dummy_base_prismatic_y_joint: limit lower=-600.2800293 upper=600.2800293 effort=4800. velocity=15. -> lower=-100.2800293 upper=100.2800293 effort=4800. velocity=15.
- joint dummy_base_revolute_z_joint: limit lower=-600.2800208 upper=600.2800208 effort=4800. velocity=15.0000002 -> lower=-100.2800208 upper=100.2800208 effort=4800. velocity=15.0000002

Commit message: improve ik

File: src/curobo/content/assets/robot/ridgeback_franka/RidgebackFranka.urdf (robot description, URDF)
Before this commit: robot RidgebackFranka, 19 links, 18 joints
Joints:
- joint dummy_base_revolute_z_joint: limit lower=-100.2800208 upper=100.2800208 effort=4800. velocity=15.0000002 -> lower=-3.2800208 upper=3.2800208 effort=4800. velocity=15.0000002

Commit message: blender motion gen pipeline init

File: src/curobo/content/assets/robot/ridgeback_franka/RidgebackFranka.urdf (robot description, URDF)
Before this commit: robot RidgebackFranka, 19 links, 18 joints
Joints:
- joint panda_joint1: limit lower=-2.9670997 upper=2.9670997 effort=5220. velocity=2.1749999 -> lower=-2.9670997 upper=2.9670997 effort=5220. velocity=12.1749999
- joint panda_joint2: limit lower=-1.8325998 upper=1.8325998 effort=5220. velocity=2.1749999 -> lower=-1.8325998 upper=1.8325998 effort=5220. velocity=12.1749999
- joint panda_joint3: limit lower=-2.9670997 upper=2.9670997 effort=5220. velocity=2.1749999 -> lower=-2.9670997 upper=2.9670997 effort=5220. velocity=12.1749999
- joint panda_joint4: limit lower=-2.9999998 upper=0.087 effort=5220. velocity=2.1749999 -> lower=-2.9999998 upper=0.087 effort=5220. velocity=12.1749999
- joint panda_joint5: limit lower=-2.9670997 upper=2.9670997 effort=720. velocity=2.6099999 -> lower=-2.9670997 upper=2.9670997 effort=720. velocity=12.6099999
- joint panda_joint6: limit lower=-0.0873 upper=2.9999998 effort=720. velocity=2.6099999 -> lower=-0.0873 upper=2.9999998 effort=720. velocity=12.6099999
- joint panda_joint7: limit lower=-2.9670997 upper=2.9670997 effort=720. velocity=2.6099999 -> lower=-2.9670997 upper=2.9670997 effort=720. velocity=12.6099999

Commit message: improve the generation

File: src/curobo/content/assets/robot/ridgeback_franka/RidgebackFranka.urdf (robot description, URDF)
Before this commit: robot RidgebackFranka, 19 links, 18 joints
Links:
- link RidgebackFranka_panda_rightfinger: geometry collision mesh filename=meshes/RidgebackFranka_panda_rightfinger_collisions.obj scale=1. 1. 1.; visual mesh filename=meshes/RidgebackFranka_panda_rightfinger_collisions.obj scale=1. 1. 1.

Commit message: fuck curobo and blender

File: src/curobo/content/assets/robot/ridgeback_franka/RidgebackFranka.urdf (robot description, URDF)
Before this commit: robot RidgebackFranka, 19 links, 18 joints
Joints:
- joint dummy_base_prismatic_x_joint: limit lower=-100.2800293 upper=100.2800293 effort=4800. velocity=15. -> lower=-30.2800293 upper=30.2800293 effort=4800. velocity=15.
- joint dummy_base_prismatic_y_joint: limit lower=-100.2800293 upper=100.2800293 effort=4800. velocity=15. -> lower=-30.2800293 upper=30.2800293 effort=4800. velocity=15.
